File: pcb/SEG-16-XXX-MDNT-L3/SEG-16-XXX-MDNT-L3.kicad_pcb (KiCad board)
At the start: 2 copper layers, 66.7 x 100 mm, 6 parts

Commit message: Updated to 0V6 changed images
Other:
- board text added: "0V6"
- board text removed: "0V5"
Changed lines of the file:
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@@
     (effects (font (size 1.5 1.5) (thickness 0.3)) (justify mirror))
   )
-  (gr_text 0V5 (at 26 30) (layer B.SilkS)
+  (gr_text 0V6 (at 26 30) (layer B.SilkS)
     (effects (font (size 1.5 1.5) (thickness 0.3)) (justify mirror))
   )
